File: pcb/ftdiy.brd (EAGLE design)
At the start: 160 x 100 mm, 2 parts, among them U1 CP2108

Commit message: Finish schematic, board and generate gerbers
Parts:
- added C1, C5: 1uF, Capacitor:CAP0603
- added C2, C3, C4: 100nF, Capacitor:CAP0603
- added D1: SP0503BAHT, TVS:SOT143
- added D10: RED, LED:0603
- added D2, D4, D7, D9: GREEN, LED:0603
- added D3, D5, D6, D8: BLUE, LED:0603
- added F1: 500mA, PTC Fuses:1206
- added JP1, JP2, JP3, JP4: PINHD-1X6, Pin Header:1X06
- added JP5: PINHD-2X3, Pin Header:2X03
- added R1: 10K Ohms, Resistor:RES0603
- added R10, R2, R3, R4, R5, R6, R7, R8, R9: 330 Ohms, Resistor:RES0603
- USB1: value USB_ID_6_SHIELD-MICRO-B-SMT -> USB-MICRO-B-SMD-FLAT-SIDE; device USB Connector:USB-UB-SMT -> USB Connector:USB-MICRO-B-SMD-FLAT-SIDE
- moved U1 42.4 mm to (24.5, 11.2)
- moved USB1 31.4 mm to (2.00, 11.1)
Connections:
- new net !P0_RX_LED: D3.1, U1.40
- new net !P0_TX_LED: D2.1, U1.41
- new net !P1_RX_LED: D5.1, U1.33
- new net !P1_TX_LED: D4.1, U1.34
- new net !P2_RX_LED: D7.1, U1.29
- new net !P2_TX_LED: D6.1, U1.30
- new net !P3_RX_LED: D9.1, U1.23
- new net !P3_TX_LED: D8.1, U1.26
- new net 3V3: C3.1, C4.1, C5.1, JP5.3, JP5.4, R1.2, U1.24, U1.39, U1.58
- new net 5V0: C1.1, C2.1, D1.4, F1.1, JP5.1, JP5.2, R10.2, R2.2, R3.2, R4.2, R5.2, R6.2, R7.2, R8.2, R9.2, U1.3, U1.60, U1.61
- new net D+: D1.2, U1.62, USB1.D+
- new net D-: D1.3, U1.63, USB1.D-
- new net GND: C1.2, C2.2, C3.2, C4.2, C5.2, D1.1, JP1.1, JP2.1, JP3.1, JP4.1, JP5.5, JP5.6, U1.2, U1.25, U1.59, U1.65, USB1.GND, USB1.SHIELD1, USB1.SHIELD2, USB1.SHIELD3, USB1.SHIELD4, USB1.SHIELD5, USB1.SHIELD6
- new net N$1: JP1.2, U1.56
- new net N$10: JP2.6, U1.45
- new net N$11: JP3.2, U1.15
- new net N$12: JP3.3, U1.16
- new net N$13: JP3.4, U1.14
- new net N$14: JP3.5, U1.13
- new net N$15: JP3.6, U1.18
- new net N$16: JP4.2, U1.1
- new net N$17: JP4.3, U1.4
- new net N$18: JP4.4, U1.6
- new net N$19: JP4.5, U1.5
- new net N$2: JP1.3, U1.57
- new net N$20: JP4.6, U1.10
- new net N$21: R1.1, U1.64
- new net N$22: D10.2, R2.1
- new net N$23: D2.2, R3.1
- new net N$24: D3.2, R4.1
- new net N$25: D4.2, R5.1
- new net N$26: D5.2, R6.1
- new net N$27: D6.2, R7.1
- new net N$28: D7.2, R8.1
- new net N$29: D8.2, R9.1
- new net N$3: JP1.4, U1.55
- new net N$30: D9.2, R10.1
- new net N$31: F1.2, USB1.VBUS
- new net N$4: JP1.5, U1.54
- new net N$5: JP1.6, U1.53
- new net N$6: JP2.2, U1.48
- new net N$7: JP2.3, U1.49
- new net N$8: JP2.4, U1.47
- new net N$9: JP2.5, U1.46
- new net PWR_LED: D10.1, U1.20
Routing:
- net 5V0: track 0.00 -> 78.2 mm, vias 0 -> 5
- net 3V3: track 0.00 -> 44.2 mm, vias 0 -> 3
- net D-: track 0.00 -> 32.9 mm, vias 0 -> 4
- net !P3_TX_LED: track 0.00 -> 32.5 mm, vias 0 -> 4
- net D+: track 0.00 -> 29.9 mm, vias 0 -> 4
- net !P3_RX_LED: track 0.00 -> 29.5 mm, vias 0 -> 4
- net N$7: track 0.00 -> 25.0 mm, vias 0 -> 2
- net !P0_RX_LED: track 0.00 -> 24.1 mm, vias 0 -> 2
- net N$6: track 0.00 -> 23.7 mm, vias 0 -> 2
- net N$1: track 0.00 -> 22.9 mm, vias 0 -> 2
- net !P1_RX_LED: track 0.00 -> 22.1 mm, vias 0 -> 2
- net N$2: track 0.00 -> 21.8 mm, vias 0 -> 1
- net !P0_TX_LED: track 0.00 -> 19.6 mm, vias 0 -> 2
- net N$8: track 0.00 -> 18.2 mm
- net N$3: track 0.00 -> 18.2 mm, vias 0 -> 1
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- added copper zone on layer 1, net GND
- added copper zone on layer 16, net GND
Other:
- board size 160 x 100 mm -> 49 x 22.5 mm
- board text added: "Designed in Portugal"
- board text added: "GND 3V3 5V0"
- board text added: "GND RXD TXD RTS CTS DTR"
- board text added: "PORT 0"
- board text added: "PORT 1"
- board text added: "PORT 2"
- board text added: "PORT 3"
- board text added: "RX0"
- board text added: "RX1"
- board text added: "RX2"
- board text added: "RX3"
- board text added: "TX0"
- board text added: "TX1"
- board text added: "TX2"
- board text added: "TX3"
- board text added: "UART 0 (3V3)"
- board text added: "UART 1 (3V3)"
- board text added: "UART 2 (3V3)"
- board text added: "UART 3 (5V0)"
