File: pcb/ftdiy.brd (EAGLE design)
At the start: 49 x 22.5 mm, 33 parts, among them U1 CP2108

Commit message: Add OSHW logo
Parts:
- added LOGO1: OSHW-LOGOM, Silkscreen:OSHW-LOGO-M
Changed lines of the file:
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@@
 <drawing>
 <settings>
-<setting alwaysvectorfont="no"/>
+<setting alwaysvectorfont="yes"/>
 <setting verticaltext="up"/>
 </settings>
@@
 <attribute name="VALUE" x="13.445" y="14.19" size="1.27" layer="27" rot="R90"/>
 </element>
+<element name="LOGO1" library="Silkscreen" package="OSHW-LOGO-M" value="OSHW-LOGOM" x="7.3" y="4.3" smashed="yes" rot="MR0"/>
 </elements>
 <signals>
